File: vca_as3360_v1/vca_as3360_v1_input_block.kicad_sch (KiCad schematic)
At the start: 42 parts, among them J4 CV1, J5 CV2, J6 IN1, J7 IN2, Q1 BC547, Q2 BC547, U3 TL072, U4 TL072

Commit message: Layout and routing first pass done
Parts:
- removed U3: TL072, Package_DIP:DIP-8_W7.62mm_Socket_LongPads, symbol Amplifier_Operational:TL072
- added R31: 10k, Resistor_SMD:R_1206_3216Metric_Pad1.30x1.75mm_HandSolder, symbol Device:R
- added R32: 100k, Resistor_SMD:R_1206_3216Metric_Pad1.30x1.75mm_HandSolder, symbol Device:R
- added U3: LM358, Package_DIP:DIP-8_W7.62mm_Socket_LongPads, symbol Amplifier_Operational:LM358
- R11, R20: value R -> 1k
- R16: value 90k -> 100k
- R25: value 90k -> 10k
Connections:
- net +12V: now also U3.8 (V+)
- net -12V: now also R32.1, U3.4 (V-); no longer R25.1
- net Linear CV 1: now also U3.1
- net Linear CV 2: now also U3.7
- net at R18.1, R19.2: now also U3.2 (-)
- net at R16.2: now also R25.1; no longer RV1.1
- net at RV2.1: now also R31.2; no longer R25.2
- net at R14.1, R17.2: now also U3.3 (+)
- net at R27.1, R28.2: now also U3.6 (-)
- net at R23.1, R26.2: now also U3.5 (+)
- new net: R31.1, R32.2
- new net: R25.2, RV1.1
Other:
- moved on the sheet: C12, C13, D4, D5, D6, J4, J5, Q2, R13, R15, R16, R20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

Commit message: Geographic rename and silkscreen cleanup
Parts:
- renumbered C14 to C101, C15 to C102, C12 to C107, C13 to C110, R15 to R1, R6 to R10, R3 to R11, R1 to R12, R19 to R16, R18 to R17, R28 to R18, R17 to R19, R25 to R2, R26 to R20, R27 to R21, R14 to R24, R12 to R26, R11 to R27, R13 to R28, R23 to R29, R16 to R3, R20 to R30, R21 to R31, R22 to R32, R30 to R4, R29 to R5, R8 to R6, R31 to R7, R24 to R8, R32 to R9, U4 to U1
