File: vca_as3360_v1/vca_as3360_v1_output_block.kicad_sch (KiCad schematic)
At the start: 11 parts, among them J2 OUT_1, J3 OUT_2, U2 TL072

Commit message: Layout and routing first pass done
Changed lines of the file:
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@@
   (junction (at 111.76 119.38) (diameter 0) (color 0 0 0 0)
   )
-  (no_connect (at 148.082 114.3))
+  (no_connect (at 147.32 114.3))
   (no_connect (at 148.59 83.82))
   (wire (pts (xy 185.42 95.885) (xy 187.96 95.885))

Commit message: Geographic rename and silkscreen cleanup
Parts:
- renumbered C10 to C108, C11 to C109, R9 to R13, R10 to R14, R7 to R15, R5 to R22, R4 to R23, R2 to R25, U2 to U4
Changed lines of the file:
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@@
   (symbol (lib_id "Device:R") (at 120.65 119.38 270) (unit 1)
     (in_bom yes) (on_board yes)
-    (property "Reference" "R10" (id 0) (at 120.65 116.84 90))
+    (property "Reference" "R14" (id 0) (at 120.65 116.84 90))
     (property "Value" "100k" (id 1) (at 120.65 121.92 90))
     (property "Footprint" "Resistor_SMD:R_1206_3216Metric_Pad1.30x1.75mm_HandSolder" (id 2) (at 120.65 117.602 90)
@@
   (symbol (lib_id "Device:R") (at 106.68 119.38 270) (unit 1)
     (in_bom yes) (on_board yes)
-    (property "Reference" "R9" (id 0) (at 106.68 116.84 90))
+    (property "Reference" "R13" (id 0) (at 106.68 116.84 90))
     (property "Value" "100k" (id 1) (at 106.68 121.92 90))
     (property "Footprint" "Resistor_SMD:R_1206_3216Metric_Pad1.30x1.75mm_HandSolder" (id 2) (at 106.68 117.602 90)
@@
   (symbol (lib_id "Device:C") (at 185.42 99.695 180) (unit 1)
     (in_bom yes) (on_board yes)
-    (property "Reference" "C11" (id 0) (at 188.341 98.5266 0)
+    (property "Reference" "C109" (id 0) (at 188.341 98.5266 0)
       (effects (font (size 1.27 1.27)) (justify right))
     )
@@
   (symbol (lib_id "Device:C") (at 185.42 92.075 180) (unit 1)
     (in_bom yes) (on_board yes)
-    (property "Reference" "C10" (id 0) (at 188.341 90.9066 0)
+    (property "Reference" "C108" (id 0) (at 188.341 90.9066 0)
       (effects (font (size 1.27 1.27)) (justify right))
     )
@@
   (symbol (lib_id "Amplifier_Operational:TL072") (at 119.38 81.28 0) (unit 1)
     (in_bom yes) (on_board yes)
-    (property "Reference" "U2" (id 0) (at 119.38 71.9582 0))
+    (property "Reference" "U4" (id 0) (at 119.38 71.9582 0))
     (property "Value" "TL072" (id 1) (at 119.38 74.2696 0))
     (property "Footprint" "Package_DIP:DIP-8_W7.62mm_Socket_LongPads" (id 2) (at 119.38 81.28 0)
@@
   (symbol (lib_id "Amplifier_Operational:TL072") (at 176.53 95.885 0) (unit 3)
     (in_bom yes) (on_board yes)
-    (property "Reference" "U2" (id 0) (at 175.4632 94.7166 0)
+    (property "Reference" "U4" (id 0) (at 175.4632 94.7166 0)
       (effects (font (size 1.27 1.27)) (justify left))
     )
@@
   (symbol (lib_id "Device:R") (at 134.62 111.76 270) (unit 1)
     (in_bom yes) (on_board yes)
-    (property "Reference" "R7" (id 0) (at 134.62 109.22 90))
+    (property "Reference" "R15" (id 0) (at 134.62 109.22 90))
     (property "Value" "1k" (id 1) (at 134.62 114.3 90))
     (property "Footprint" "Resistor_SMD:R_1206_3216Metric_Pad1.30x1.75mm_HandSolder" (id 2) (at 134.62 109.982 90)
@@
   (symbol (lib_id "Device:R") (at 106.68 88.9 270) (unit 1)
     (in_bom yes) (on_board yes)
-    (property "Reference" "R4" (id 0) (at 106.68 86.36 90))
+    (property "Reference" "R23" (id 0) (at 106.68 86.36 90))
     (property "Value" "100k" (id 1) (at 106.68 91.44 90))
     (property "Footprint" "Resistor_SMD:R_1206_3216Metric_Pad1.30x1.75mm_HandSolder" (id 2) (at 106.68 87.122 90)
@@
   (symbol (lib_id "Device:R") (at 134.62 81.28 270) (unit 1)
     (in_bom yes) (on_board yes)
-    (property "Reference" "R2" (id 0) (at 134.62 78.74 90))
+    (property "Reference" "R25" (id 0) (at 134.62 78.74 90))
     (property "Value" "1k" (id 1) (at 134.62 83.82 90))
     (property "Footprint" "Resistor_SMD:R_1206_3216Metric_Pad1.30x1.75mm_HandSolder" (id 2) (at 134.62 79.502 90)
@@
   (symbol (lib_id "Device:R") (at 120.65 88.9 270) (unit 1)
     (in_bom yes) (on_board yes)
-    (property "Reference" "R5" (id 0) (at 120.65 86.36 90))
+    (property "Reference" "R22" (id 0) (at 120.65 86.36 90))
     (property "Value" "100k" (id 1) (at 120.65 91.44 90))
     (property "Footprint" "Resistor_SMD:R_1206_3216Metric_Pad1.30x1.75mm_HandSolder" (id 2) (at 120.65 87.122 90)
@@
   (symbol (lib_id "Amplifier_Operational:TL072") (at 119.38 111.76 0) (unit 2)
     (in_bom yes) (on_board yes)
-    (property "Reference" "U2" (id 0) (at 119.38 102.4382 0))
+    (property "Reference" "U4" (id 0) (at 119.38 102.4382 0))
     (property "Value" "TL072" (id 1) (at 119.38 104.7496 0))
     (property "Footprint" "Package_DIP:DIP-8_W7.62mm_Socket_LongPads" (id 2) (at 119.38 111.76 0)
