File: vca_as3360_v1/vca_as3360_v1_vco_block.kicad_sch (KiCad schematic)
At the start: 6 parts, among them U1 AS3360

Commit message: Layout and routing first pass done
Parts:
- removed C8, C9: 10nF, Capacitor_SMD:C_1206_3216Metric_Pad1.33x1.80mm_HandSolder, symbol Device:C

Commit message: Geographic rename and silkscreen cleanup
Parts:
- renumbered C6 to C104, C3 to C105, C7 to C106, U1 to U2
Changed lines of the file:
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@@
   (symbol (lib_id "Device:C") (at 141.605 87.63 0) (unit 1)
     (in_bom yes) (on_board yes) (fields_autoplaced)
-    (property "Reference" "C7" (id 0) (at 144.526 86.7215 0)
+    (property "Reference" "C106" (id 0) (at 144.526 86.7215 0)
       (effects (font (size 1.27 1.27)) (justify left))
     )
@@
   (symbol (lib_id "Device:C") (at 141.605 53.975 180) (unit 1)
     (in_bom yes) (on_board yes) (fields_autoplaced)
-    (property "Reference" "C3" (id 0) (at 138.684 54.8835 0)
+    (property "Reference" "C105" (id 0) (at 138.684 54.8835 0)
       (effects (font (size 1.27 1.27)) (justify left))
     )
@@
   (symbol (lib_id "Audio:AS3360") (at 141.986 129.54 0) (unit 2)
     (in_bom yes) (on_board yes) (fields_autoplaced)
-    (property "Reference" "U1" (id 0) (at 144.0054 117.9535 0)
+    (property "Reference" "U2" (id 0) (at 144.0054 117.9535 0)
       (effects (font (size 1.27 1.27)) (justify left))
     )
@@
   (symbol (lib_id "Audio:AS3360") (at 141.605 69.85 0) (unit 1)
     (in_bom yes) (on_board yes) (fields_autoplaced)
-    (property "Reference" "U1" (id 0) (at 143.6244 58.2635 0)
+    (property "Reference" "U2" (id 0) (at 143.6244 58.2635 0)
       (effects (font (size 1.27 1.27)) (justify left))
     )
@@
   (symbol (lib_id "Device:C") (at 125.73 76.2 0) (unit 1)
     (in_bom yes) (on_board yes) (fields_autoplaced)
-    (property "Reference" "C6" (id 0) (at 128.651 75.2915 0)
+    (property "Reference" "C104" (id 0) (at 128.651 75.2915 0)
       (effects (font (size 1.27 1.27)) (justify left))
     )
